File: Alumirror-right/Alumirror-matrix.kicad_sch (KiCad schematic)
At the start: 45 parts, among them K11 PG1350, K12 PG1350, K13 PG1350, K14 PG1350, K15 PG1350, K16 PG1350, K21 PG1350, K22 PG1350, K23 PG1350, K24 PG1350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

Commit message: Updated Row 3 diode placement
Connections:
- net Col6: now also K16.1, K26.1; no longer K16.2, K26.2
- net at D26.2 (A): now also K26.2; no longer K26.1
- net at D16.2 (A): now also K16.2; no longer K16.1
Changed lines of the file:
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@@
 		(lib_id "Switch:SW_Push")
 		(at 217.17 81.28 0)
+		(mirror y)
 		(unit 1)
 		(exclude_from_sim no)
@@
 		(lib_id "Switch:SW_Push")
 		(at 217.17 53.34 0)
-		(unit 1)
-		(exclude_from_sim no)
+		(mirror y)
+		(unit 1)
+		(exclude_from_sim no)
