File: Alumirror-matrix.kicad_sch (KiCad schematic)
At the start: 41 parts, among them K11 PG1350, K12 PG1350, K13 PG1350, K14 PG1350, K15 PG1350, K16 PG1350, K21 PG1350, K22 PG1350, K23 PG1350, K24 PG1350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

Commit message: Various tweaks
Parts:
- removed R17: 0R, Project Library:R_2010_5025Metric_Mod, symbol Device:R
Connections:
- net Col2: now also K31.1
Changed lines of the file:
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@@
 	(wire
 		(pts
-			(xy 115.57 82.55) (xy 115.57 99.06)
+			(xy 199.39 43.18) (xy 199.39 71.12)
 		)
 		(stroke
@@
 	(wire
 		(pts
-			(xy 199.39 43.18) (xy 199.39 71.12)
+			(xy 199.39 71.12) (xy 199.39 74.93)
 		)
 		(stroke
@@
 	(wire
 		(pts
-			(xy 199.39 71.12) (xy 199.39 74.93)
-		)
-		(stroke
-			(width 0)
-			(type default)
-		)
-	)
-	(wire
-		(pts
-			(xy 115.57 71.12) (xy 115.57 74.93)
+			(xy 115.57 71.12) (xy 115.57 99.06)
 		)
 		(stroke
@@
 					(unit 1)
 				)
-			)
-		)
-	)
-	(symbol
-		(lib_id "Device:R")
-		(at 115.57 78.74 0)
-		(unit 1)
-		(exclude_from_sim no)
-		(in_bom yes)
-		(on_board yes)
-		(dnp no)
-		(fields_autoplaced yes)
-		(property "Reference" "R17"
-			(at 118.11 77.4699 0)
-			(effects
-				(font
-					(size 1.27 1.27)
-				)
-				(justify left)
-			)
-		)
-		(property "Value" "0R"
-			(at 118.11 80.0099 0)
-			(effects
-				(font
-					(size 1.27 1.27)
-				)
-				(justify left)
-			)
-		)
-		(property "Footprint" "Project Library:R_2010_5025Metric_Mod"
-			(at 113.792 78.74 90)
-			(effects
-				(font
-					(size 1.27 1.27)
-				)
-				(hide yes)
-			)
-		)
-		(property "Datasheet" "~"
-			(at 115.57 78.74 0)
-			(effects
-				(font
-					(size 1.27 1.27)
-				)
-				(hide yes)
-			)
-		)
-		(property "Description" "Resistor"
-			(at 115.57 78.74 0)
-			(effects
-				(font
-					(size 1.27 1.27)
-				)
-				(hide yes)
-			)
-		)
-		(pin "1"
-		)
-		(pin "2"
-		)
-		(instances
-			(project "Alumirror"
-				(path "/52f043ac-ccff-4c85-bc10-2db9d3c9e3f3/ba0213d9-9934-4194-9bec-bf394cd27126"
-					(reference "R17")
-					(unit 1)
-				)
