File: Alufo-matrix.kicad_sch (KiCad schematic)
At the start: 54 parts, among them K11 PG1350, K12 PG1350, K13 PG1350, K14 PG1350, K15 PG1350, K16 PG1350, K21 PG1350, K22 PG1350, K23 PG1350, K24 PG1350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

Commit message: Change project name from Alumirror to Alufo
Since it is likely that the left and right hand PCBs will be split, there won’t actually be much mirroring going on (also most split keyboards are mirrored left to right, so that not particularly special or unique!). Instead the name will emphasise the slight flying saucer look of the PCB with Al(uminium) + UFO = Alufo.
Other:
- title: Alumirror  -> Alufo 
Changed lines of the file:
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@@
 	(paper "A4")
 	(title_block
-		(title "Alumirror ")
+		(title "Alufo ")
 		(rev "0.1")
 		(company "bgkendall")
@@
 		)
 		(instances
-			(project "Alumirror"
+			(project "Alufo"
 				(path "/52f043ac-ccff-4c85-bc10-2db9d3c9e3f3/ba0213d9-9934-4194-9bec-bf394cd27126"
 					(reference "D45")
@@
 		)
 		(instances
-			(project "Alumirror"
+			(project "Alufo"
 				(path "/52f043ac-ccff-4c85-bc10-2db9d3c9e3f3/ba0213d9-9934-4194-9bec-bf394cd27126"
 					(reference "K24")
@@
 		)
 		(instances
-			(project "Alumirror"
+			(project "Alufo"
 				(path "/52f043ac-ccff-4c85-bc10-2db9d3c9e3f3/ba0213d9-9934-4194-9bec-bf394cd27126"
 					(reference "K23")
@@
 		)
 		(instances
-			(project "Alumirror"
+			(project "Alufo"
 				(path "/52f043ac-ccff-4c85-bc10-2db9d3c9e3f3/ba0213d9-9934-4194-9bec-bf394cd27126"
 					(reference "K33")
@@
 		)
 		(instances
-			(project "Alumirror"
+			(project "Alufo"
 				(path "/52f043ac-ccff-4c85-bc10-2db9d3c9e3f3/ba0213d9-9934-4194-9bec-bf394cd27126"
 					(reference "K14")
@@
 		)
 		(instances
-			(project "Alumirror"
+			(project "Alufo"
 				(path "/52f043ac-ccff-4c85-bc10-2db9d3c9e3f3/ba0213d9-9934-4194-9bec-bf394cd27126"
 					(reference "R13")
@@
 		)
 		(instances
-			(project "Alumirror"
+			(project "Alufo"
 				(path "/52f043ac-ccff-4c85-bc10-2db9d3c9e3f3/ba0213d9-9934-4194-9bec-bf394cd27126"
 					(reference "K34")
@@
 		)
 		(instances
-			(project "Alumirror"
+			(project "Alufo"
 				(path "/52f043ac-ccff-4c85-bc10-2db9d3c9e3f3/ba0213d9-9934-4194-9bec-bf394cd27126"
 					(reference "K36")
@@
 		)
 		(instances
-			(project "Alumirror"
+			(project "Alufo"
 				(path "/52f043ac-ccff-4c85-bc10-2db9d3c9e3f3/ba0213d9-9934-4194-9bec-bf394cd27126"
 					(reference "D36")
@@
 		)
 		(instances
-			(project "Alumirror"
+			(project "Alufo"
 				(path "/52f043ac-ccff-4c85-bc10-2db9d3c9e3f3/ba0213d9-9934-4194-9bec-bf394cd27126"
 					(reference "R11")
@@
 		)
 		(instances
-			(project "Alumirror"
+			(project "Alufo"
 				(path "/52f043ac-ccff-4c85-bc10-2db9d3c9e3f3/ba0213d9-9934-4194-9bec-bf394cd27126"
 					(reference "D12")
@@
 		)
 		(instances
-			(project "Alumirror"
+			(project "Alufo"
 				(path "/52f043ac-ccff-4c85-bc10-2db9d3c9e3f3/ba0213d9-9934-4194-9bec-bf394cd27126"
 					(reference "D31")
@@
 		)
 		(instances
-			(project "Alumirror"
+			(project "Alufo"
 				(path "/52f043ac-ccff-4c85-bc10-2db9d3c9e3f3/ba0213d9-9934-4194-9bec-bf394cd27126"
 					(reference "D43")
@@
 		)
 		(instances
-			(project "Alumirror"
+			(project "Alufo"
 				(path "/52f043ac-ccff-4c85-bc10-2db9d3c9e3f3/ba0213d9-9934-4194-9bec-bf394cd27126"
 					(reference "K11")
@@
 		)
 		(instances
-			(project "Alumirror"
+			(project "Alufo"
 				(path "/52f043ac-ccff-4c85-bc10-2db9d3c9e3f3/ba0213d9-9934-4194-9bec-bf394cd27126"
 					(reference "R19")
@@
 		)
 		(instances
-			(project "Alumirror"
+			(project "Alufo"
 				(path "/52f043ac-ccff-4c85-bc10-2db9d3c9e3f3/ba0213d9-9934-4194-9bec-bf394cd27126"
 					(reference "R16")
@@
 		)
 		(instances
-			(project "Alumirror"
+			(project "Alufo"
 				(path "/52f043ac-ccff-4c85-bc10-2db9d3c9e3f3/ba0213d9-9934-4194-9bec-bf394cd27126"
 					(reference "R12")
@@
 		)
 		(instances
-			(project "Alumirror"
+			(project "Alufo"
 				(path "/52f043ac-ccff-4c85-bc10-2db9d3c9e3f3/ba0213d9-9934-4194-9bec-bf394cd27126"
 					(reference "K42")
@@
 		)
 		(instances
-			(project "Alumirror"
+			(project "Alufo"
 				(path "/52f043ac-ccff-4c85-bc10-2db9d3c9e3f3/ba0213d9-9934-4194-9bec-bf394cd27126"
 					(reference "R14")
@@
 		)
 		(instances
-			(project "Alumirror"
+			(project "Alufo"
 				(path "/52f043ac-ccff-4c85-bc10-2db9d3c9e3f3/ba0213d9-9934-4194-9bec-bf394cd27126"
 					(reference "K31")
@@
 		)
 		(instances
-			(project "Alumirror"
+			(project "Alufo"
 				(path "/52f043ac-ccff-4c85-bc10-2db9d3c9e3f3/ba0213d9-9934-4194-9bec-bf394cd27126"
 					(reference "D46")
@@
 		)
 		(instances
-			(project "Alumirror"
+			(project "Alufo"
 				(path "/52f043ac-ccff-4c85-bc10-2db9d3c9e3f3/ba0213d9-9934-4194-9bec-bf394cd27126"
 					(reference "D15")
@@
 		)
 		(instances
-			(project "Alumirror"
+			(project "Alufo"
 				(path "/52f043ac-ccff-4c85-bc10-2db9d3c9e3f3/ba0213d9-9934-4194-9bec-bf394cd27126"
 					(reference "K41")
@@
 		)
 		(instances
-			(project "Alumirror"
+			(project "Alufo"
 				(path "/52f043ac-ccff-4c85-bc10-2db9d3c9e3f3/ba0213d9-9934-4194-9bec-bf394cd27126"
 					(reference "K21")
@@
 		)
 		(instances
-			(project "Alumirror"
+			(project "Alufo"
 				(path "/52f043ac-ccff-4c85-bc10-2db9d3c9e3f3/ba0213d9-9934-4194-9bec-bf394cd27126"
 					(reference "D26")
@@
 		)
 		(instances
-			(project "Alumirror"
+			(project "Alufo"
 				(path "/52f043ac-ccff-4c85-bc10-2db9d3c9e3f3/ba0213d9-9934-4194-9bec-bf394cd27126"
 					(reference "K15")
@@
 		)
 		(instances
-			(project "Alumirror"
+			(project "Alufo"
 				(path "/52f043ac-ccff-4c85-bc10-2db9d3c9e3f3/ba0213d9-9934-4194-9bec-bf394cd27126"
 					(reference "K32")
@@
 		)
 		(instances
-			(project "Alumirror"
+			(project "Alufo"
 				(path "/52f043ac-ccff-4c85-bc10-2db9d3c9e3f3/ba0213d9-9934-4194-9bec-bf394cd27126"
 					(reference "D32")
@@
 		)
 		(instances
-			(project "Alumirror"
+			(project "Alufo"
 				(path "/52f043ac-ccff-4c85-bc10-2db9d3c9e3f3/ba0213d9-9934-4194-9bec-bf394cd27126"
 					(reference "K12")
@@
 		)
 		(instances
-			(project "Alumirror"
+			(project "Alufo"
 				(path "/52f043ac-ccff-4c85-bc10-2db9d3c9e3f3/ba0213d9-9934-4194-9bec-bf394cd27126"
 					(reference "D33")
@@
 		)
 		(instances
-			(project "Alumirror"
+			(project "Alufo"
 				(path "/52f043ac-ccff-4c85-bc10-2db9d3c9e3f3/ba0213d9-9934-4194-9bec-bf394cd27126"
 					(reference "D16")
@@
 		)
 		(instances
-			(project "Alumirror"
+			(project "Alufo"
 				(path "/52f043ac-ccff-4c85-bc10-2db9d3c9e3f3/ba0213d9-9934-4194-9bec-bf394cd27126"
 					(reference "D34")
@@
 		)
 		(instances
-			(project "Alumirror"
+			(project "Alufo"
 				(path "/52f043ac-ccff-4c85-bc10-2db9d3c9e3f3/ba0213d9-9934-4194-9bec-bf394cd27126"
 					(reference "K35")
@@
 		)
 		(instances
-			(project "Alumirror"
+			(project "Alufo"
 				(path "/52f043ac-ccff-4c85-bc10-2db9d3c9e3f3/ba0213d9-9934-4194-9bec-bf394cd27126"
 					(reference "K25")
@@
 		)
 		(instances
-			(project "Alumirror"
+			(project "Alufo"
 				(path "/52f043ac-ccff-4c85-bc10-2db9d3c9e3f3/ba0213d9-9934-4194-9bec-bf394cd27126"
 					(reference "D41")
@@
 		)
 		(instances
-			(project "Alumirror"
+			(project "Alufo"
 				(path "/52f043ac-ccff-4c85-bc10-2db9d3c9e3f3/ba0213d9-9934-4194-9bec-bf394cd27126"
 					(reference "D21")
@@
 		)
 		(instances
-			(project "Alumirror"
+			(project "Alufo"
 				(path "/52f043ac-ccff-4c85-bc10-2db9d3c9e3f3/ba0213d9-9934-4194-9bec-bf394cd27126"
 					(reference "D13")
@@
 		)
 		(instances
-			(project "Alumirror"
+			(project "Alufo"
 				(path "/52f043ac-ccff-4c85-bc10-2db9d3c9e3f3/ba0213d9-9934-4194-9bec-bf394cd27126"
 					(reference "D23")
@@
 		)
 		(instances
-			(project "Alumirror"
+			(project "Alufo"
 				(path "/52f043ac-ccff-4c85-bc10-2db9d3c9e3f3/ba0213d9-9934-4194-9bec-bf394cd27126"
 					(reference "D25")
@@
 		)
 		(instances
-			(project "Alumirror"
+			(project "Alufo"
 				(path "/52f043ac-ccff-4c85-bc10-2db9d3c9e3f3/ba0213d9-9934-4194-9bec-bf394cd27126"
 					(reference "R18")
@@
 		)
 		(instances
-			(project "Alumirror"
+			(project "Alufo"
 				(path "/52f043ac-ccff-4c85-bc10-2db9d3c9e3f3/ba0213d9-9934-4194-9bec-bf394cd27126"
 					(reference "D11")
@@
 		)
 		(instances
-			(project "Alumirror"
+			(project "Alufo"
 				(path "/52f043ac-ccff-4c85-bc10-2db9d3c9e3f3/ba0213d9-9934-4194-9bec-bf394cd27126"
 					(reference "R17")
@@
 		)
 		(instances
-			(project "Alumirror"
+			(project "Alufo"
 				(path "/52f043ac-ccff-4c85-bc10-2db9d3c9e3f3/ba0213d9-9934-4194-9bec-bf394cd27126"
 					(reference "D24")
@@
 		)
 		(instances
-			(project "Alumirror"
+			(project "Alufo"
 				(path "/52f043ac-ccff-4c85-bc10-2db9d3c9e3f3/ba0213d9-9934-4194-9bec-bf394cd27126"
 					(reference "K22")
@@
 		)
 		(instances
-			(project "Alumirror"
+			(project "Alufo"
 				(path "/52f043ac-ccff-4c85-bc10-2db9d3c9e3f3/ba0213d9-9934-4194-9bec-bf394cd27126"
 					(reference "R20")
@@
 		)
 		(instances
-			(project "Alumirror"
+			(project "Alufo"
 				(path "/52f043ac-ccff-4c85-bc10-2db9d3c9e3f3/ba0213d9-9934-4194-9bec-bf394cd27126"
 					(reference "K13")
@@
 		)
 		(instances
-			(project "Alumirror"
+			(project "Alufo"
 				(path "/52f043ac-ccff-4c85-bc10-2db9d3c9e3f3/ba0213d9-9934-4194-9bec-bf394cd27126"
 					(reference "D42")
@@
 		)
 		(instances
-			(project "Alumirror"
+			(project "Alufo"
 				(path "/52f043ac-ccff-4c85-bc10-2db9d3c9e3f3/ba0213d9-9934-4194-9bec-bf394cd27126"
 					(reference "K26")
@@
 		)
 		(instances
-			(project "Alumirror"
+			(project "Alufo"
 				(path "/52f043ac-ccff-4c85-bc10-2db9d3c9e3f3/ba0213d9-9934-4194-9bec-bf394cd27126"
 					(reference "D44")
@@
 		)
 		(instances
-			(project "Alumirror"
+			(project "Alufo"
 				(path "/52f043ac-ccff-4c85-bc10-2db9d3c9e3f3/ba0213d9-9934-4194-9bec-bf394cd27126"
 					(reference "R15")
@@
 		)
 		(instances
-			(project "Alumirror"
+			(project "Alufo"
 				(path "/52f043ac-ccff-4c85-bc10-2db9d3c9e3f3/ba0213d9-9934-4194-9bec-bf394cd27126"
 					(reference "D35")
@@
 		)
 		(instances
-			(project "Alumirror"
+			(project "Alufo"
 				(path "/52f043ac-ccff-4c85-bc10-2db9d3c9e3f3/ba0213d9-9934-4194-9bec-bf394cd27126"
 					(reference "D22")
@@
 		)
 		(instances
-			(project "Alumirror"
+			(project "Alufo"
 				(path "/52f043ac-ccff-4c85-bc10-2db9d3c9e3f3/ba0213d9-9934-4194-9bec-bf394cd27126"
 					(reference "K16")
@@
 		)
 		(instances
-			(project "Alumirror"
+			(project "Alufo"
 				(path "/52f043ac-ccff-4c85-bc10-2db9d3c9e3f3/ba0213d9-9934-4194-9bec-bf394cd27126"
 					(reference "D14")
