File: Alufo.kicad_sch (KiCad schematic)
At the start: 42 parts, among them J1 USB_C_Receptacle_USB2.0_16P_2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, J2 USB_C_Receptacle_USB2.0_16P_2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, J3 USB_C_Receptacle_USB2.0_16P_2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, J4 USB_C_Receptacle_USB2.0_16P_2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, SW10 BOOT, U1 CH552T, U2 CH552T, U3 USBLC6-2P6, U4 USBLC6-2P6, U5 USBLC6-2P6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

Commit message: Change project name from Alumirror to Alufo
Since it is likely that the left and right hand PCBs will be split, there won’t actually be much mirroring going on (also most split keyboards are mirrored left to right, so that not particularly special or unique!). Instead the name will emphasise the slight flying saucer look of the PCB with Al(uminium) + UFO = Alufo.
Other:
- sheet Matrix: file Alumirror-matrix.kicad_sch -> Alufo-matrix.kicad_sch
- title: Alumirror  -> Alufo 
