File: Left/Alufo.kicad_sch (KiCad schematic)
At the start: 42 parts, among them J1 USB_C_Receptacle_USB2.0_16P_2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, J2 USB_C_Receptacle_USB2.0_16P_2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, J3 USB_C_Receptacle_USB2.0_16P_2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, J4 USB_C_Receptacle_USB2.0_16P_2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, SW10 BOOT, U1 CH552T, U2 CH552T, U3 USBLC6-2P6, U4 USBLC6-2P6, U5 USBLC6-2P6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

Commit message: Remove righthand components from lefthand board
Parts:
- removed C2, C4: 100nF, Capacitor_SMD:C_0603_1608Metric, symbol Device:C
- removed D2: PMEG2010EA, Diode_SMD:D_SOD-323, symbol Device:D_Schottky
- removed F2: 500mA, Fuse:Fuse_0603_1608Metric, symbol Device:Polyfuse_Small
- removed FB2: FerriteBead, Inductor_SMD:L_0805_2012Metric, symbol Device:FerriteBead
- removed H6: MountingHole, Project Library:MountingHole_2.2mm_M2_SMD_Solder_Nut, symbol Mechanical:MountingHole
- removed J2, J4: USB_C_Receptacle_USB2.0_16P_2SH, Project Library:USB_C_Receptacle_HRO_TYPE-C-31-M-12, symbol Project Library:USB_C_Receptacle_USB2.0_16P_2SH
- removed NT2: NetTie_2, Project Library:NetTie-2_SMD_Pad0.2mm, symbol Device:NetTie_2
- removed R2, R4: 5k1, Resistor_SMD:R_0603_1608Metric, symbol Device:R
- removed R6: 5k1-20k, Resistor_SMD:R_0603_1608Metric, symbol Device:R
- removed U2: CH552T, Package_SO:TSSOP-20_4.4x6.5mm_P0.65mm, symbol Project Library:MCU_CH552T_TSSOP-20
- removed U4, U6: USBLC6-2P6, Project Library:SOT-666_Mod, symbol Power_Protection:USBLC6-2P6
Connections:
- no-connect marks 33 -> 17
