File: Left/Alufo-matrix.kicad_sch (KiCad schematic)
At the start: 54 parts, among them K11 PG1350, K12 PG1350, K13 PG1350, K14 PG1350, K15 PG1350, K16 PG1350, K21 PG1350, K22 PG1350, K23 PG1350, K24 PG1350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

Commit message: Remove righthand components from lefthand board
Parts:
- removed D41, D42, D43, D44, D45, D46: 1N4148, Project Library:D_SOD-123, symbol Device:D
- removed K41: PG1350_1½U, Project Library:SW_choc_v1_HS_CPG135001S30_1layer_1.5u, symbol Switch:SW_Push
- removed K42: PG1350/SKQUCAA010, Project Library:SW_choc_v1_HS_nav_CPG135001S30_SKQUCAA010_1layer_1u_1, symbol Project Library:SW_SP5T

Commit message: Align upper 0Ω resistors as on righthand, remove R11
Parts:
- removed R11: 0R, Project Library:R_2010_5025Metric_Mod, symbol Device:R
Connections:
- net Col1T is gone; now on net Col1: K21.1, K31.1
- net Col2RT: no longer names the net of K32.1, R17.2
- net Col3RT: no longer names the net of K33.1, R18.2
- net Col4RT: no longer names the net of K34.1, R19.2
Changed lines of the file:
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@@
-	(wire
-		(pts
-			(xy 87.63 64.77) (xy 87.63 81.28)
-		)
-		(stroke
-			(width 0)
-			(type default)
-		)
-	)
 	(wire
 		(pts
@@
 	(wire
 		(pts
-			(xy 87.63 53.34) (xy 87.63 57.15)
+			(xy 87.63 53.34) (xy 87.63 81.28)
 		)
 		(stroke
@@
 		)
 	)
-	(global_label "Col3RT"
-		(shape input)
-		(at 166.37 93.98 0)
+	(global_label "Col6T"
+		(shape input)
+		(at 227.33 81.28 0)
 		(fields_autoplaced yes)
 		(effects
@@
 		)
 		(property "Intersheetrefs" "${INTERSHEET_REFS}"
-			(at 175.8865 93.98 0)
+			(at 235.5765 81.28 0)
 			(effects
 				(font
@@
 		)
 	)
-	(global_label "Col2RT"
-		(shape input)
-		(at 138.43 93.98 0)
+	(global_label "Col5L"
+		(shape input)
+		(at 199.39 43.18 0)
 		(fields_autoplaced yes)
 		(effects
@@
 		)
 		(property "Intersheetrefs" "${INTERSHEET_REFS}"
-			(at 147.9465 93.98 0)
+			(at 207.697 43.18 0)
 			(effects
 				(font
@@
 		)
 	)
-	(global_label "Col4RT"
-		(shape input)
-		(at 194.31 99.06 0)
+	(global_label "Col4R"
+		(shape input)
+		(at 171.45 60.96 0)
 		(fields_autoplaced yes)
 		(effects
@@
 		)
 		(property "Intersheetrefs" "${INTERSHEET_REFS}"
-			(at 203.8265 99.06 0)
+			(at 179.9989 60.96 0)
 			(effects
 				(font
@@
 		)
 	)
-	(global_label "Col6T"
-		(shape input)
-		(at 227.33 81.28 0)
+	(global_label "Row1"
+		(shape input)
+		(at 68.58 60.96 180)
+		(fields_autoplaced yes)
+		(effects
+			(font
+				(size 1.27 1.27)
+			)
+			(justify right)
+		)
+		(property "Intersheetrefs" "${INTERSHEET_REFS}"
+			(at 60.6358 60.96 0)
+			(effects
+				(font
+					(size 1.27 1.27)
+				)
+				(justify right)
+				(hide yes)
+			)
+		)
+	)
+	(global_label "Col3L"
+		(shape input)
+		(at 143.51 38.1 0)
 		(fields_autoplaced yes)
 		(effects
@@
 		)
 		(property "Intersheetrefs" "${INTERSHEET_REFS}"
-			(at 235.5765 81.28 0)
+			(at 151.817 38.1 0)
 			(effects
 				(font
@@
 		)
 	)
-	(global_label "Col5L"
-		(shape input)
-		(at 199.39 43.18 0)
+	(global_label "Col5T"
+		(shape input)
+		(at 139.7 147.32 0)
 		(fields_autoplaced yes)
 		(effects
@@
 		)
 		(property "Intersheetrefs" "${INTERSHEET_REFS}"
-			(at 207.697 43.18 0)
+			(at 147.9465 147.32 0)
 			(effects
 				(font
@@
 		)
 	)
-	(global_label "Col4R"
-		(shape input)
-		(at 171.45 60.96 0)
+	(global_label "Col2R"
+		(shape input)
+		(at 115.57 60.96 0)
 		(fields_autoplaced yes)
 		(effects
@@
 		)
 		(property "Intersheetrefs" "${INTERSHEET_REFS}"
-			(at 179.9989 60.96 0)
+			(at 124.1189 60.96 0)
 			(effects
 				(font
@@
 		)
 	)
-	(global_label "Row1"
-		(shape input)
-		(at 68.58 60.96 180)
+	(global_label "Col4L"
+		(shape input)
+		(at 171.45 38.1 0)
+		(fields_autoplaced yes)
+		(effects
+			(font
+				(size 1.27 1.27)
+			)
+			(justify left)
+		)
+		(property "Intersheetrefs" "${INTERSHEET_REFS}"
+			(at 179.757 38.1 0)
+			(effects
+				(font
+					(size 1.27 1.27)
+				)
+				(justify left)
+				(hide yes)
+			)
+		)
+	)
+	(global_label "Col6"
+		(shape input)
+		(at 227.33 53.34 0)
+		(fields_autoplaced yes)
+		(effects
+			(font
+				(size 1.27 1.27)
+			)
+			(justify left)
+		)
+		(property "Intersheetrefs" "${INTERSHEET_REFS}"
+			(at 234.6089 53.34 0)
+			(effects
+				(font
+					(size 1.27 1.27)
+				)
+				(justify left)
+				(hide yes)
+			)
+		)
+	)
+	(global_label "Row2"
+		(shape input)
+		(at 68.58 88.9 180)
 		(fields_autoplaced yes)
 		(effects
@@
 		)
 		(property "Intersheetrefs" "${INTERSHEET_REFS}"
-			(at 60.6358 60.96 0)
+			(at 60.6358 88.9 0)
 			(effects
 				(font
@@
 				)
 				(justify right)
-				(hide yes)
-			)
-		)
-	)
-	(global_label "Col3L"
-		(shape input)
-		(at 143.51 38.1 0)
-		(fields_autoplaced yes)
-		(effects
-			(font
-				(size 1.27 1.27)
-			)
-			(justify left)
-		)
-		(property "Intersheetrefs" "${INTERSHEET_REFS}"
-			(at 151.817 38.1 0)
-			(effects
-				(font
-					(size 1.27 1.27)
-				)
-				(justify left)
-				(hide yes)
-			)
-		)
-	)
-	(global_label "Col5T"
-		(shape input)
-		(at 139.7 147.32 0)
-		(fields_autoplaced yes)
-		(effects
-			(font
-				(size 1.27 1.27)
-			)
-			(justify left)
-		)
-		(property "Intersheetrefs" "${INTERSHEET_REFS}"
-			(at 147.9465 147.32 0)
-			(effects
-				(font
-					(size 1.27 1.27)
-				)
-				(justify left)
-				(hide yes)
-			)
-		)
-	)
-	(global_label "Col2R"
-		(shape input)
-		(at 115.57 60.96 0)
-		(fields_autoplaced yes)
-		(effects
-			(font
-				(size 1.27 1.27)
-			)
-			(justify left)
-		)
-		(property "Intersheetrefs" "${INTERSHEET_REFS}"
-			(at 124.1189 60.96 0)
-			(effects
-				(font
-					(size 1.27 1.27)
-				)
-				(justify left)
-				(hide yes)
-			)
-		)
-	)
-	(global_label "Col4L"
-		(shape input)
-		(at 171.45 38.1 0)
-		(fields_autoplaced yes)
-		(effects
-			(font
-				(size 1.27 1.27)
-			)
-			(justify left)
-		)
-		(property "Intersheetrefs" "${INTERSHEET_REFS}"
-			(at 179.757 38.1 0)
-			(effects
-				(font
-					(size 1.27 1.27)
-				)
-				(justify left)
-				(hide yes)
-			)
-		)
-	)
-	(global_label "Col6"
-		(shape input)
-		(at 227.33 53.34 0)
-		(fields_autoplaced yes)
-		(effects
-			(font
-				(size 1.27 1.27)
-			)
-			(justify left)
-		)
-		(property "Intersheetrefs" "${INTERSHEET_REFS}"
-			(at 234.6089 53.34 0)
-			(effects
-				(font
-					(size 1.27 1.27)
-				)
-				(justify left)
-				(hide yes)
-			)
-		)
-	)
-	(global_label "Row2"
-		(shape input)
-		(at 68.58 88.9 180)
-		(fields_autoplaced yes)
-		(effects
-			(font
-				(size 1.27 1.27)
-			)
-			(justify right)
-		)
-		(property "Intersheetrefs" "${INTERSHEET_REFS}"
-			(at 60.6358 88.9 0)
-			(effects
-				(font
-					(size 1.27 1.27)
-				)
-				(justify right)
-				(hide yes)
-			)
-		)
-	)
-	(global_label "Col1T"
-		(shape input)
-		(at 110.49 99.06 0)
-		(fields_autoplaced yes)
-		(effects
-			(font
-				(size 1.27 1.27)
-			)
-			(justify left)
-		)
-		(property "Intersheetrefs" "${INTERSHEET_REFS}"
-			(at 118.7365 99.06 0)
-			(effects
-				(font
-					(size 1.27 1.27)
-				)
-				(justify left)
 				(hide yes)
 			)
@@
 					(unit 1)
 				)
-			)
-		)
-	)
-	(symbol
-		(lib_id "Device:R")
-		(at 87.63 60.96 0)
-		(unit 1)
-		(exclude_from_sim no)
-		(in_bom yes)
-		(on_board yes)
-		(dnp no)
-		(property "Reference" "R11"
-			(at 90.17 59.6899 0)
-			(effects
-				(font
-					(size 1.27 1.27)
-				)
-				(justify left)
-			)
-		)
-		(property "Value" "0R"
-			(at 90.17 62.2299 0)
-			(effects
-				(font
-					(size 1.27 1.27)
-				)
-				(justify left)
-			)
-		)
-		(property "Footprint" "Project Library:R_2010_5025Metric_Mod"
-			(at 85.852 60.96 90)
-			(effects
-				(font
-					(size 1.27 1.27)
-				)
-				(hide yes)
-			)
-		)
-		(property "Datasheet" "~"
-			(at 87.63 60.96 0)
-			(effects
-				(font
-					(size 1.27 1.27)
-				)
-				(hide yes)
-			)
-		)
-		(property "Description" "Resistor"
-			(at 87.63 60.96 0)
-			(effects
-				(font
-					(size 1.27 1.27)
-				)
-				(hide yes)
-			)
-		)
-		(pin "1"
-		)
-		(pin "2"
-		)
-		(instances
-			(project "Alufo"
-				(path "/52f043ac-ccff-4c85-bc10-2db9d3c9e3f3/ba0213d9-9934-4194-9bec-bf394cd27126"
-					(reference "R11")
-					(unit 1)
-				)

Commit message: Remove lower 0Ω resistors
Parts:
- removed R17, R18, R19, R20: 0R, Project Library:R_2010_5025Metric_Mod, symbol Device:R
Connections:
- net Col2R is gone; now on an unnamed net: K22.1, R12.2
- net Col3R is gone; now on an unnamed net: K23.1, R13.2
- net Col4R is gone; now on an unnamed net: K24.1, R14.2
- net Col5R is gone; now on net Col5T: K25.1, R15.2

Commit message: Remove “L” from column labels
Connections:
- net Col2L renamed Col2
- net Col3L renamed Col3
- net Col4L renamed Col4
- net Col5L renamed Col5
Changed lines of the file:
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@@
+	)
+	(junction
+		(at 227.33 81.28)
+		(diameter 0)
+		(color 0 0 0 0)
 	)
 	(junction
@@
 	(wire
 		(pts
+			(xy 227.33 81.28) (xy 227.33 83.82)
+		)
+		(stroke
+			(width 0)
+			(type default)
+		)
+	)
+	(wire
+		(pts
 			(xy 166.37 83.82) (xy 166.37 93.98)
 		)
@@
 	(wire
 		(pts
+			(xy 100.33 50.8) (xy 100.33 60.96)
+		)
+		(stroke
+			(width 0)
+			(type default)
+		)
+	)
+	(wire
+		(pts
+			(xy 143.51 66.04) (xy 143.51 83.82)
+		)
+		(stroke
+			(width 0)
+			(type default)
+		)
+	)
+	(wire
+		(pts
+			(xy 110.49 71.12) (xy 115.57 71.12)
+		)
+		(stroke
+			(width 0)
+			(type default)
+		)
+	)
+	(wire
+		(pts
+			(xy 120.65 50.8) (xy 100.33 50.8)
+		)
+		(stroke
+			(width 0)
+			(type default)
+		)
+	)
+	(wire
+		(pts
+			(xy 110.49 43.18) (xy 115.57 43.18)
+		)
+		(stroke
+			(width 0)
+			(type default)
+		)
+	)
+	(wire
+		(pts
+			(xy 115.57 43.18) (xy 115.57 46.99)
+		)
+		(stroke
+			(width 0)
+			(type default)
+		)
+	)
+	(wire
+		(pts
+			(xy 171.45 38.1) (xy 171.45 41.91)
+		)
+		(stroke
+			(width 0)
+			(type default)
+		)
+	)
+	(wire
+		(pts
+			(xy 100.33 106.68) (xy 128.27 106.68)
+		)
+		(stroke
+			(width 0)
+			(type default)
+		)
+	)
+	(wire
+		(pts
+			(xy 199.39 54.61) (xy 199.39 71.12)
+		)
+		(stroke
+			(width 0)
+			(type default)
+		)
+	)
+	(wire
+		(pts
 			(xy 222.25 81.28) (xy 227.33 81.28)
-		)
-		(stroke
-			(width 0)
-			(type default)
-		)
-	)
-	(wire
-		(pts
-			(xy 100.33 50.8) (xy 100.33 60.96)
-		)
-		(stroke
-			(width 0)
-			(type default)
-		)
-	)
-	(wire
-		(pts
-			(xy 143.51 66.04) (xy 143.51 83.82)
-		)
-		(stroke
-			(width 0)
-			(type default)
-		)
-	)
-	(wire
-		(pts
-			(xy 110.49 71.12) (xy 115.57 71.12)
-		)
-		(stroke
-			(width 0)
-			(type default)
-		)
-	)
-	(wire
-		(pts
-			(xy 120.65 50.8) (xy 100.33 50.8)
-		)
-		(stroke
-			(width 0)
-			(type default)
-		)
-	)
-	(wire
-		(pts
-			(xy 110.49 43.18) (xy 115.57 43.18)
-		)
-		(stroke
-			(width 0)
-			(type default)
-		)
-	)
-	(wire
-		(pts
-			(xy 115.57 43.18) (xy 115.57 46.99)
-		)
-		(stroke
-			(width 0)
-			(type default)
-		)
-	)
-	(wire
-		(pts
-			(xy 171.45 38.1) (xy 171.45 41.91)
-		)
-		(stroke
-			(width 0)
-			(type default)
-		)
-	)
-	(wire
-		(pts
-			(xy 100.33 106.68) (xy 128.27 106.68)
-		)
-		(stroke
-			(width 0)
-			(type default)
-		)
-	)
-	(wire
-		(pts
-			(xy 199.39 54.61) (xy 199.39 71.12)
 		)
 		(stroke
@@
 	(global_label "Col6T"
 		(shape input)
-		(at 227.33 81.28 0)
+		(at 227.33 83.82 270)
+		(fields_autoplaced yes)
+		(effects
+			(font
+				(size 1.27 1.27)
+			)
+			(justify right)
+		)
+		(property "Intersheetrefs" "${INTERSHEET_REFS}"
+			(at 227.33 92.0665 90)
+			(effects
+				(font
+					(size 1.27 1.27)
+				)
+				(justify right)
+				(hide yes)
+			)
+		)
+	)
+	(global_label "Col5"
+		(shape input)
+		(at 199.39 43.18 0)
 		(fields_autoplaced yes)
 		(effects
@@
 		)
 		(property "Intersheetrefs" "${INTERSHEET_REFS}"
-			(at 235.5765 81.28 0)
+			(at 206.6689 43.18 0)
 			(effects
 				(font
@@
 		)
 	)
-	(global_label "Col5L"
-		(shape input)
-		(at 199.39 43.18 0)
+	(global_label "Row1"
+		(shape input)
+		(at 68.58 60.96 180)
+		(fields_autoplaced yes)
+		(effects
+			(font
+				(size 1.27 1.27)
+			)
+			(justify right)
+		)
+		(property "Intersheetrefs" "${INTERSHEET_REFS}"
+			(at 60.6358 60.96 0)
+			(effects
+				(font
+					(size 1.27 1.27)
+				)
+				(justify right)
+				(hide yes)
+			)
+		)
+	)
+	(global_label "Col3"
+		(shape input)
+		(at 143.51 38.1 0)
 		(fields_autoplaced yes)
 		(effects
@@
 		)
 		(property "Intersheetrefs" "${INTERSHEET_REFS}"
-			(at 207.697 43.18 0)
+			(at 150.7889 38.1 0)
 			(effects
 				(font
@@
 		)
 	)
-	(global_label "Row1"
-		(shape input)
-		(at 68.58 60.96 180)
+	(global_label "Col5T"
+		(shape input)
+		(at 139.7 147.32 0)
+		(fields_autoplaced yes)
+		(effects
+			(font
+				(size 1.27 1.27)
+			)
+			(justify left)
+		)
+		(property "Intersheetrefs" "${INTERSHEET_REFS}"
+			(at 147.9465 147.32 0)
+			(effects
+				(font
+					(size 1.27 1.27)
+				)
+				(justify left)
+				(hide yes)
+			)
+		)
+	)
+	(global_label "Col4"
+		(shape input)
+		(at 171.45 38.1 0)
+		(fields_autoplaced yes)
+		(effects
+			(font
+				(size 1.27 1.27)
+			)
+			(justify left)
+		)
+		(property "Intersheetrefs" "${INTERSHEET_REFS}"
+			(at 178.7289 38.1 0)
+			(effects
+				(font
+					(size 1.27 1.27)
+				)
+				(justify left)
+				(hide yes)
+			)
+		)
+	)
+	(global_label "Col6"
+		(shape input)
+		(at 227.33 53.34 0)
+		(fields_autoplaced yes)
+		(effects
+			(font
+				(size 1.27 1.27)
+			)
+			(justify left)
+		)
+		(property "Intersheetrefs" "${INTERSHEET_REFS}"
+			(at 234.6089 53.34 0)
+			(effects
+				(font
+					(size 1.27 1.27)
+				)
+				(justify left)
+				(hide yes)
+			)
+		)
+	)
+	(global_label "Row2"
+		(shape input)
+		(at 68.58 88.9 180)
 		(fields_autoplaced yes)
 		(effects
@@
 		)
 		(property "Intersheetrefs" "${INTERSHEET_REFS}"
-			(at 60.6358 60.96 0)
+			(at 60.6358 88.9 0)
 			(effects
 				(font
@@
 		)
 	)
-	(global_label "Col3L"
-		(shape input)
-		(at 143.51 38.1 0)
+	(global_label "Col2"
+		(shape input)
+		(at 115.57 43.18 0)
 		(fields_autoplaced yes)
 		(effects
@@
 		)
 		(property "Intersheetrefs" "${INTERSHEET_REFS}"
-			(at 151.817 38.1 0)
-			(effects
-				(font
-					(size 1.27 1.27)
-				)
-				(justify left)
-				(hide yes)
-			)
-		)
-	)
-	(global_label "Col5T"
-		(shape input)
-		(at 139.7 147.32 0)
-		(fields_autoplaced yes)
-		(effects
-			(font
-				(size 1.27 1.27)
-			)
-			(justify left)
-		)
-		(property "Intersheetrefs" "${INTERSHEET_REFS}"
-			(at 147.9465 147.32 0)
-			(effects
-				(font
-					(size 1.27 1.27)
-				)
-				(justify left)
-				(hide yes)
-			)
-		)
-	)
-	(global_label "Col4L"
-		(shape input)
-		(at 171.45 38.1 0)
-		(fields_autoplaced yes)
-		(effects
-			(font
-				(size 1.27 1.27)
-			)
-			(justify left)
-		)
-		(property "Intersheetrefs" "${INTERSHEET_REFS}"
-			(at 179.757 38.1 0)
-			(effects
-				(font
-					(size 1.27 1.27)
-				)
-				(justify left)
-				(hide yes)
-			)
-		)
-	)
-	(global_label "Col6"
-		(shape input)
-		(at 227.33 53.34 0)
-		(fields_autoplaced yes)
-		(effects
-			(font
-				(size 1.27 1.27)
-			)
-			(justify left)
-		)
-		(property "Intersheetrefs" "${INTERSHEET_REFS}"
-			(at 234.6089 53.34 0)
-			(effects
-				(font
-					(size 1.27 1.27)
-				)
-				(justify left)
-				(hide yes)
-			)
-		)
-	)
-	(global_label "Row2"
-		(shape input)
-		(at 68.58 88.9 180)
-		(fields_autoplaced yes)
-		(effects
-			(font
-				(size 1.27 1.27)
-			)
-			(justify right)
-		)
-		(property "Intersheetrefs" "${INTERSHEET_REFS}"
-			(at 60.6358 88.9 0)
-			(effects
-				(font
-					(size 1.27 1.27)
-				)
-				(justify right)
-				(hide yes)
-			)
-		)
-	)
-	(global_label "Col2L"
-		(shape input)
-		(at 115.57 43.18 0)
-		(fields_autoplaced yes)
-		(effects
-			(font
-				(size 1.27 1.27)
-			)
-			(justify left)
-		)
-		(property "Intersheetrefs" "${INTERSHEET_REFS}"
-			(at 123.877 43.18 0)
-			(effects
-				(font
+			(at 122.8489 43.18 0)
+			(effects
+				(font

Commit message: Manually add cutouts for 2010 resistors
Using middle-layer cutouts defined in the footprint no longer works as the resistors are now vertically aligned in relation to each rather than a set distance from the switch sockets.
Parts:
- R12, R13, R14, R15, R16: footprint Project Library:R_2010_5025Metric_Mod -> Resistor_SMD:R_2010_5025Metric
Changed lines of the file:
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@@
 			)
 		)
-		(property "Footprint" "Project Library:R_2010_5025Metric_Mod"
+		(property "Footprint" "Resistor_SMD:R_2010_5025Metric"
 			(at 141.732 45.72 90)
 			(effects
@@
 			)
 		)
-		(property "Footprint" "Project Library:R_2010_5025Metric_Mod"
+		(property "Footprint" "Resistor_SMD:R_2010_5025Metric"
 			(at 225.552 60.96 90)
 			(effects
@@
 			)
 		)
-		(property "Footprint" "Project Library:R_2010_5025Metric_Mod"
+		(property "Footprint" "Resistor_SMD:R_2010_5025Metric"
 			(at 113.792 50.8 90)
 			(effects
@@
 			)
 		)
-		(property "Footprint" "Project Library:R_2010_5025Metric_Mod"
+		(property "Footprint" "Resistor_SMD:R_2010_5025Metric"
 			(at 169.672 45.72 90)
 			(effects
@@
 			)
 		)
-		(property "Footprint" "Project Library:R_2010_5025Metric_Mod"
+		(property "Footprint" "Resistor_SMD:R_2010_5025Metric"
 			(at 197.612 50.8 90)
 			(effects
