File: Left/Alufo.kicad_pcb (KiCad board)
At the start: 2 copper layers, 139.7 x 88.9 mm, 67 parts, among them J1 USB_C_Receptacle_USB2.0_16P_2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, J3 USB_C_Receptacle_USB2.0_16P_2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, K11 PG1350, K12 PG1350, K13 PG1350, K14 PG1350, K15 PG1350, K16 PG1350, K21 PG1350, K22 PG1350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

Commit message: Add fun logo on lefthand board
Other:
- board text added: "${PROJECTNAME} v${PCB_REVISION} • ${AUTHOR}"
- board text removed: "${AUTHOR}"
