File: Right/Alufo.kicad_sch (KiCad schematic)
At the start: 22 parts, among them J2 USB_C_Receptacle_USB2.0_16P_2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, J4 USB_C_Receptacle_USB2.0_16P_2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, SW10 BOOT, U2 CH552T, U4 USBLC6-2P6, U6 USBLC6-2P6

Commit message: Renumber previously common components
Parts:
- renumbered L10 to L2, R10 to R8, SW10 to SW2
Changed lines of the file:
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@@
 		(dnp no)
 		(fields_autoplaced yes)
-		(property "Reference" "L10"
+		(property "Reference" "L2"
 			(at 167.9575 115.57 0)
 			(effects
@@
 			(project ""
 				(path "/52f043ac-ccff-4c85-bc10-2db9d3c9e3f3"
-					(reference "L10")
+					(reference "L2")
 					(unit 1)
 				)
@@
 		(on_board yes)
 		(dnp no)
-		(property "Reference" "R10"
+		(property "Reference" "R8"
 			(at 179.07 118.11 90)
 			(effects
@@
 			(project "Alufo"
 				(path "/52f043ac-ccff-4c85-bc10-2db9d3c9e3f3"
-					(reference "R10")
+					(reference "R8")
 					(unit 1)
 				)
@@
 		(dnp no)
 		(fields_autoplaced yes)
-		(property "Reference" "SW10"
+		(property "Reference" "SW2"
 			(at 172.72 101.6 0)
 			(effects
@@
 			(project "Alufo"
 				(path "/52f043ac-ccff-4c85-bc10-2db9d3c9e3f3"
-					(reference "SW10")
-					(unit 1)
-				)
+					(reference "SW2")
+					(unit 1)
+				)

Commit message: Fix boot access hole location
Because the lefthand side PCB will become the base for the righthand board (and vice versa), and because the boot button is no longer centred, the hole in the base to allow access to the button must be on the opposite side of the centreline to that button. This means the access hole needs to be a separate component and the boot switch footprint no longer needs a central hole.
Parts:
- added H6: BootAccess, MountingHole:MountingHole_2.5mm, symbol Mechanical:MountingHole
Changed lines of the file:
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@@
+	)
+	(symbol
+		(lib_id "Mechanical:MountingHole")
+		(at 177.8 176.53 0)
+		(unit 1)
+		(exclude_from_sim yes)
+		(in_bom no)
+		(on_board yes)
+		(dnp no)
+		(fields_autoplaced yes)
+		(property "Reference" "H6"
+			(at 180.34 175.2599 0)
+			(effects
+				(font
+					(size 1.27 1.27)
+				)
+				(justify left)
+			)
+		)
+		(property "Value" "BootAccess"
+			(at 180.34 177.7999 0)
+			(effects
+				(font
+					(size 1.27 1.27)
+				)
+				(justify left)
+			)
+		)
+		(property "Footprint" "MountingHole:MountingHole_2.5mm"
+			(at 177.8 176.53 0)
+			(effects
+				(font
+					(size 1.27 1.27)
+				)
+				(hide yes)
+			)
+		)
+		(property "Datasheet" "~"
+			(at 177.8 176.53 0)
+			(effects
+				(font
+					(size 1.27 1.27)
+				)
+				(hide yes)
+			)
+		)
+		(property "Description" "Mounting Hole without connection"
+			(at 177.8 176.53 0)
+			(effects
+				(font
+					(size 1.27 1.27)
+				)
+				(hide yes)
+			)
+		)
+		(instances
+			(project "Alufo"
+				(path "/52f043ac-ccff-4c85-bc10-2db9d3c9e3f3"
+					(reference "H6")
+					(unit 1)
+				)
+			)
+		)
 	)
 	(symbol
