File: PCB Right/Alufo-matrix.kicad_sch (KiCad schematic)
At the start: 63 parts, among them K11 PG1350, K12 PG1350, K13 PG1350, K14 PG1350, K15 PG1350, K16 PG1350, K21 PG1350, K22 PG1350, K23 PG1350, K24 PG1350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

Commit message: Apply similar changes to right PCB
Parts:
- removed R11, R12, R13, R14, R15: 0R, Resistor_SMD:R_2010_5025Metric, symbol Device:R
Connections:
- net Col1T is gone; now on net Col1: K21.1, K41.1
- net Col2T is gone; now on net Col2: D42.2 (A), K22.1, K32.1
- net Col3T is gone; now on net Col3: D43.2 (A), K23.1, K33.1
- net Col4T is gone; now on net Col4: D44.2 (A), K24.1, K34.1
- net Col5T is gone; now on net Col5: D45.2 (A), K25.1, K35.1
- net Row1: no longer D16.1 (K)
