File: PCB Left/Alufo.kicad_sch (KiCad schematic)
At the start: 35 parts, among them J1 USB_C_Receptacle_USB2.0_16P_2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, J3 USB_C_Receptacle_USB2.0_16P_2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, SW1 BOOT, U1 CH552T, U3 USBLC6-2P6, U5 USBLC6-2P6

Commit message: Correct LCSC part number for USB port
Reviewed all other parts
Parts:
- J1, J3: LCSC C165948 -> C5143397
Changed lines of the file:
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@@
 			)
 		)
-		(property "LCSC" "C165948"
+		(property "LCSC" "C5143397"
 			(at 46.99 166.37 0)
 			(effects
@@
 			)
 		)
-		(property "LCSC" "C165948"
+		(property "LCSC" "C5143397"
 			(at 46.99 100.33 0)
 			(effects

Commit message: Remove 0Ω resistor (R9) on VCC line
Rework some routing around USB port.
Remove keep out areas from switch to allow additional ground connections.
Use personal SOD-323 footprint.
Parts:
- removed NT1: NetTie_2, Project_Library:NetTie-2_SMD_Pad0.2mm, symbol Device:NetTie_2
- removed R9: 0R, Resistor_SMD:R_2010_5025Metric, symbol Device:R
- D1: footprint Diode_SMD:D_SOD-323 -> BGK_Kicad:D_SOD-323
Connections:
- net VCC' is gone; now on net VCC: J3.A4 (VBUS), J3.A9 (VBUS), J3.B4 (VBUS), J3.B9 (VBUS), U5.5 (VBUS)
- net SHIELD: now also FB1.1
- net USB+: now also R5.1
- net at J1.S2 (SHIELD): no longer FB1.1
- no-connect marks 15 -> 16
Other:
- moved on the sheet: FB1

Commit message: Remove lefthand R12
Can route Col1, Col2 and Row2 around each other without needing jumper on Col2.
Col1 and Col2 pins on MCU swapped.
Connections:
- net Col1: now also U1.4 (P1.6); no longer U1.5 (P1.7)
- net Col2: now also U1.5 (P1.7); no longer U1.4 (P1.6)
Changed lines of the file:
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@@
 	(global_label "Col1"
 		(shape input)
+		(at 38.1 50.8 180)
+		(fields_autoplaced yes)
+		(effects
+			(font
+				(size 1.27 1.27)
+			)
+			(justify right)
+		)
+		(property "Intersheetrefs" "${INTERSHEET_REFS}"
+			(at 30.8211 50.8 0)
+			(effects
+				(font
+					(size 1.27 1.27)
+				)
+				(justify right)
+				(hide yes)
+			)
+		)
+	)
+	(global_label "TX_P"
+		(shape input)
+		(at 125.73 179.07 0)
+		(fields_autoplaced yes)
+		(effects
+			(font
+				(size 1.27 1.27)
+			)
+			(justify left)
+		)
+		(property "Intersheetrefs" "${INTERSHEET_REFS}"
+			(at 133.1299 179.07 0)
+			(effects
+				(font
+					(size 1.27 1.27)
+				)
+				(justify left)
+				(hide yes)
+			)
+		)
+	)
+	(global_label "Col5"
+		(shape input)
+		(at 60.96 63.5 0)
+		(fields_autoplaced yes)
+		(effects
+			(font
+				(size 1.27 1.27)
+			)
+			(justify left)
+		)
+		(property "Intersheetrefs" "${INTERSHEET_REFS}"
+			(at 68.2389 63.5 0)
+			(effects
+				(font
+					(size 1.27 1.27)
+				)
+				(justify left)
+				(hide yes)
+			)
+		)
+	)
+	(global_label "USB+"
+		(shape input)
+		(at 60.96 58.42 0)
+		(fields_autoplaced yes)
+		(effects
+			(font
+				(size 1.27 1.27)
+			)
+			(justify left)
+		)
+		(property "Intersheetrefs" "${INTERSHEET_REFS}"
+			(at 69.3276 58.42 0)
+			(effects
+				(font
+					(size 1.27 1.27)
+				)
+				(justify left)
+				(hide yes)
+			)
+		)
+	)
+	(global_label "Row3"
+		(shape input)
+		(at 38.1 60.96 180)
+		(fields_autoplaced yes)
+		(effects
+			(font
+				(size 1.27 1.27)
+			)
+			(justify right)
+		)
+		(property "Intersheetrefs" "${INTERSHEET_REFS}"
+			(at 30.1558 60.96 0)
+			(effects
+				(font
+					(size 1.27 1.27)
+				)
+				(justify right)
+				(hide yes)
+			)
+		)
+	)
+	(global_label "USB_P-"
+		(shape input)
+		(at 125.73 115.57 0)
+		(fields_autoplaced yes)
+		(effects
+			(font
+				(size 1.27 1.27)
+			)
+			(justify left)
+		)
+		(property "Intersheetrefs" "${INTERSHEET_REFS}"
+			(at 136.3352 115.57 0)
+			(effects
+				(font
+					(size 1.27 1.27)
+				)
+				(justify left)
+				(hide yes)
+			)
+		)
+	)
+	(global_label "LED"
+		(shape input)
+		(at 60.96 50.8 0)
+		(fields_autoplaced yes)
+		(effects
+			(font
+				(size 1.27 1.27)
+			)
+			(justify left)
+		)
+		(property "Intersheetrefs" "${INTERSHEET_REFS}"
+			(at 67.3923 50.8 0)
+			(effects
+				(font
+					(size 1.27 1.27)
+				)
+				(justify left)
+				(hide yes)
+			)
+		)
+	)
+	(global_label "Row2"
+		(shape input)
+		(at 38.1 58.42 180)
+		(fields_autoplaced yes)
+		(effects
+			(font
+				(size 1.27 1.27)
+			)
+			(justify right)
+		)
+		(property "Intersheetrefs" "${INTERSHEET_REFS}"
+			(at 30.1558 58.42 0)
+			(effects
+				(font
+					(size 1.27 1.27)
+				)
+				(justify right)
+				(hide yes)
+			)
+		)
+	)
+	(global_label "Col3"
+		(shape input)
+		(at 38.1 48.26 180)
+		(fields_autoplaced yes)
+		(effects
+			(font
+				(size 1.27 1.27)
+			)
+			(justify right)
+		)
+		(property "Intersheetrefs" "${INTERSHEET_REFS}"
+			(at 30.8211 48.26 0)
+			(effects
+				(font
+					(size 1.27 1.27)
+				)
+				(justify right)
+				(hide yes)
+			)
+		)
+	)
+	(global_label "Col2"
+		(shape input)
 		(at 38.1 53.34 180)
 		(fields_autoplaced yes)
@@
 			(effects
 				(font
-					(size 1.27 1.27)
-				)
-				(justify right)
-				(hide yes)
-			)
-		)
-	)
-	(global_label "TX_P"
-		(shape input)
-		(at 125.73 179.07 0)
-		(fields_autoplaced yes)
-		(effects
-			(font
-				(size 1.27 1.27)
-			)
-			(justify left)
-		)
-		(property "Intersheetrefs" "${INTERSHEET_REFS}"
-			(at 133.1299 179.07 0)
-			(effects
-				(font
-					(size 1.27 1.27)
-				)
-				(justify left)
-				(hide yes)
-			)
-		)
-	)
-	(global_label "Col5"
-		(shape input)
-		(at 60.96 63.5 0)
-		(fields_autoplaced yes)
-		(effects
-			(font
-				(size 1.27 1.27)
-			)
-			(justify left)
-		)
-		(property "Intersheetrefs" "${INTERSHEET_REFS}"
-			(at 68.2389 63.5 0)
-			(effects
-				(font
-					(size 1.27 1.27)
-				)
-				(justify left)
-				(hide yes)
-			)
-		)
-	)
-	(global_label "USB+"
-		(shape input)
-		(at 60.96 58.42 0)
-		(fields_autoplaced yes)
-		(effects
-			(font
-				(size 1.27 1.27)
-			)
-			(justify left)
-		)
-		(property "Intersheetrefs" "${INTERSHEET_REFS}"
-			(at 69.3276 58.42 0)
-			(effects
-				(font
-					(size 1.27 1.27)
-				)
-				(justify left)
-				(hide yes)
-			)
-		)
-	)
-	(global_label "Row3"
-		(shape input)
-		(at 38.1 60.96 180)
-		(fields_autoplaced yes)
-		(effects
-			(font
-				(size 1.27 1.27)
-			)
-			(justify right)
-		)
-		(property "Intersheetrefs" "${INTERSHEET_REFS}"
-			(at 30.1558 60.96 0)
-			(effects
-				(font
-					(size 1.27 1.27)
-				)
-				(justify right)
-				(hide yes)
-			)
-		)
-	)
-	(global_label "USB_P-"
-		(shape input)
-		(at 125.73 115.57 0)
-		(fields_autoplaced yes)
-		(effects
-			(font
-				(size 1.27 1.27)
-			)
-			(justify left)
-		)
-		(property "Intersheetrefs" "${INTERSHEET_REFS}"
-			(at 136.3352 115.57 0)
-			(effects
-				(font
-					(size 1.27 1.27)
-				)
-				(justify left)
-				(hide yes)
-			)
-		)
-	)
-	(global_label "LED"
-		(shape input)
-		(at 60.96 50.8 0)
-		(fields_autoplaced yes)
-		(effects
-			(font
-				(size 1.27 1.27)
-			)
-			(justify left)
-		)
-		(property "Intersheetrefs" "${INTERSHEET_REFS}"
-			(at 67.3923 50.8 0)
-			(effects
-				(font
-					(size 1.27 1.27)
-				)
-				(justify left)
-				(hide yes)
-			)
-		)
-	)
-	(global_label "Row2"
-		(shape input)
-		(at 38.1 58.42 180)
-		(fields_autoplaced yes)
-		(effects
-			(font
-				(size 1.27 1.27)
-			)
-			(justify right)
-		)
-		(property "Intersheetrefs" "${INTERSHEET_REFS}"
-			(at 30.1558 58.42 0)
-			(effects
-				(font
-					(size 1.27 1.27)
-				)
-				(justify right)
-				(hide yes)
-			)
-		)
-	)
-	(global_label "Col3"
-		(shape input)
-		(at 38.1 48.26 180)
-		(fields_autoplaced yes)
-		(effects
-			(font
-				(size 1.27 1.27)
-			)
-			(justify right)
-		)
-		(property "Intersheetrefs" "${INTERSHEET_REFS}"
-			(at 30.8211 48.26 0)
-			(effects
-				(font
-					(size 1.27 1.27)
-				)
-				(justify right)
-				(hide yes)
-			)
-		)
-	)
-	(global_label "Col2"
-		(shape input)
-		(at 38.1 50.8 180)
-		(fields_autoplaced yes)
-		(effects
-			(font
-				(size 1.27 1.27)
-			)
-			(justify right)
-		)
-		(property "Intersheetrefs" "${INTERSHEET_REFS}"
-			(at 30.8211 50.8 0)
-			(effects
-				(font

Commit message: Update LCSC part number for USB ports
Also hide LCSC numbers erroneously showing in schematic.
Parts:
- J1, J3: LCSC C5143397 -> C2681552
Changed lines of the file:
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@@
 			)
 		)
-		(property "LCSC" "C5143397"
+		(property "LCSC" "C2681552"
 			(at 46.99 166.37 0)
 			(effects
@@
 			)
 		)
-		(property "LCSC" "C5143397"
+		(property "LCSC" "C2681552"
 			(at 46.99 100.33 0)
 			(effects

Commit message: Add shield connectors
The USB ports will now be connected to the aluminium PCB core. This is done using a 0.6mm diameter wire. One end of the wire will be soldered to a pad on the PCB and the other will pass through a hole to friction fit against the aluminium core.

Also, R9, the 0Ω resistor on the lefthand VCC line has returned to allow a more direct ground route between the USB port and the MCU. However it is now a smaller 0805 size resistor.
Parts:
- removed FB1: FerriteBead, Inductor_SMD:L_0805_2012Metric, symbol Device:FerriteBead
- added J5, J7: Shield_Connection, Project_Library:Shield_Connector, symbol Connector_Generic:Conn_01x01
- added R9: 0R, Resistor_SMD:R_0805_2012Metric, symbol Device:R
Connections:
- net VCC: now also R9.1; no longer J3.A4 (VBUS), J3.A9 (VBUS), J3.B4 (VBUS), J3.B9 (VBUS), U5.5 (VBUS)
- net at J3.S1 (SHIELD): now also J7.1 (Pin_1)
- net at J1.S3 (SHIELD): now also J5.1 (Pin_1)
- net SHIELD: no longer names the net of J3.S3 (SHIELD)
- net SHIELD: no longer J1.S1 (SHIELD)
- new net VCC': J3.A4 (VBUS), J3.A9 (VBUS), J3.B4 (VBUS), J3.B9 (VBUS), R9.2, U5.5 (VBUS)

Commit message: Add shield connection to H3 (lower middle mounting hole)
Parts:
- added J9: Shield_Connection, Project_Library:Shield_Connector, symbol Connector_Generic:Conn_01x01
- H3: footprint Project_Library:MountingHole_2.2mm_M2_SMD_Solder_Nut -> Project_Library:MountingHole_2.2mm_M2_SMD_Solder_Nut_Pad; symbol Mechanical:MountingHole -> Mechanical:MountingHole_Pad
Connections:
- new net: H3.1, J9.1 (Pin_1)
Other:
- moved on the sheet: H1, H2
